File: motherboard.sch (KiCad schematic (older format))
At the start: 141 parts, among them J1 USB_C_Receptacle_USB2.0, J10 Power input, J11 Bed, J12 Hotend, J13 X_LIMIT, J14 Y_LIMIT, J15 Z_LIMIT, J16 E_LIMIT, J2 I2C, J3 EXP1, J4 EXP2, J5 BFP_touch, J6 FAN1, J7 FAN2, J8 BED_TEMP, J9 HOTEND_TEMP, M1 NEMA17, M2 NEMA17, M3 NEMA17, M4 NEMA17, Q1 BC847, Q2 BC847, Q3 AO3400A, Q4 AO3400A, Q5 APM4010, Q6 APM4010, U1 MP1584, U2 STM32F103C8Tx, U3 CH340G, U4 A4988, U5 A4988, U6 A4988, U7 A4988, Y1 8MHz, Y2 12MHz

Commit message: new pcb and fix schematic
Parts:
- removed C48: 10n, Capacitor_SMD:C_0603_1608Metric_Pad1.08x0.95mm_HandSolder, symbol Device:C
- removed J16: E_LIMIT, Connector_JST:JST_EH_B2B-EH-A_1x02_P2.50mm_Vertical, symbol Connector_Generic:Conn_01x02
- removed J2: I2C, Connector_JST:JST_EH_B4B-EH-A_1x04_P2.50mm_Vertical, symbol Connector_Generic:Conn_01x04
- removed J3: EXP1, Connector_IDC:IDC-Header_2x05_P2.54mm_Vertical, symbol ICs:IDC10
- removed J4: EXP2, Connector_IDC:IDC-Header_2x05_P2.54mm_Vertical, symbol ICs:IDC10
- removed J5: BFP_touch, Connector_JST:JST_EH_B6B-EH-A_1x06_P2.50mm_Vertical, symbol Connector_Generic:Conn_01x06
- removed J7: FAN2, Connector_JST:JST_EH_B2B-EH-A_1x02_P2.50mm_Vertical, symbol Connector_Generic:Conn_01x02
- removed JP1: Jumper, Jumper:SolderJumper-2_P1.3mm_Open_TrianglePad1.0x1.5mm, symbol Device:Jumper
- removed Q4: AO3400A, Package_TO_SOT_SMD:SOT-23, symbol Transistor_FET:AO3400A
- removed U3: CH340G, Package_SO:SOIC-16_3.9x9.9mm_P1.27mm, symbol Interface_USB:CH340G
- removed Y2: 12MHz, Crystal:Crystal_SMD_HC49-SD, symbol Device:Crystal_Small
- added C48: 10u, Capacitor_Tantalum_SMD:CP_EIA-3528-21_Kemet-B_Pad1.50x2.35mm_HandSolder, symbol Device:CP
- added C49, C50: 0u1, Capacitor_SMD:C_0603_1608Metric_Pad1.08x0.95mm_HandSolder, symbol Device:C
- added D5: D_Schottky, Diode_SMD:D_SOD-323_HandSoldering, symbol Device:D_Schottky
- added D6, D7: LED, LED_SMD:LED_0603_1608Metric_Pad1.05x0.95mm_HandSolder, symbol Device:LED
- added J2: SWD, Connector_PinHeader_2.54mm:PinHeader_1x05_P2.54mm_Vertical, symbol Connector_Generic:Conn_01x05
- added J3: EXP, Connector_IDC:IDC-Header_2x07_P2.54mm_Vertical, symbol Connector_Generic:Conn_02x07_Odd_Even
- added J5: Conn_01x03, Connector_JST:JST_XH_B3B-XH-A_1x03_P2.50mm_Vertical, symbol Connector_Generic:Conn_01x03
- added J7: Conn_02x03_Odd_Even, Connector_PinHeader_2.54mm:PinHeader_2x03_P2.54mm_Vertical, symbol Connector_Generic:Conn_02x03_Odd_Even
- added JP2: BOOT, Jumper:SolderJumper-2_P1.3mm_Open_TrianglePad1.0x1.5mm, symbol Jumper:Jumper_2_Open
- added R52, R53: 10k, Resistor_SMD:R_0603_1608Metric_Pad0.98x0.95mm_HandSolder, symbol Device:R
- added R54: 1k, Resistor_SMD:R_0603_1608Metric_Pad0.98x0.95mm_HandSolder, symbol Device:R
- added U3: AMS1117-3.3, Package_TO_SOT_SMD:SOT-223-3_TabPin2, symbol Regulator_Linear:AMS1117-3.3
- added U8: USBLC6-2SC6, Package_TO_SOT_SMD:SOT-23-6, symbol Power_Protection:USBLC6-2SC6
- C10: value 1u -> 0u1
- C11: value 10n -> 0u1
- C12, C3: footprint Capacitor_THT:CP_Radial_D6.3mm_P2.50mm -> Capacitor_Tantalum_SMD:CP_EIA-3528-21_Kemet-B_Pad1.50x2.35mm_HandSolder
- C7, C9: value 22p -> 10u; footprint Capacitor_SMD:C_0603_1608Metric_Pad1.08x0.95mm_HandSolder -> Capacitor_SMD:C_0805_2012Metric_Pad1.18x1.45mm_HandSolder
- J10, J11, J12: footprint TerminalBlock_4Ucon:TerminalBlock_4Ucon_1x02_P3.50mm_Horizontal -> TerminalBlock:TerminalBlock_bornier-2_P5.08mm
- J13, J14, J15, J8, J9: footprint Connector_JST:JST_EH_B2B-EH-A_1x02_P2.50mm_Vertical -> Connector_JST:JST_XH_B2B-XH-A_1x02_P2.50mm_Vertical
- J6: value FAN1 -> FAN; footprint Connector_JST:JST_EH_B2B-EH-A_1x02_P2.50mm_Vertical -> Connector_JST:JST_XH_B2B-XH-A_1x02_P2.50mm_Vertical
- M1, M2, M3, M4: footprint Connector_JST:JST_EH_B4B-EH-A_1x04_P2.50mm_Vertical -> Connector_JST:JST_XH_B4B-XH-A_1x04_P2.50mm_Vertical
- R21, R23, R25, R27: footprint Resistor_SMD:R_0603_1608Metric_Pad0.98x0.95mm_HandSolder -> Potentiometer_SMD:Potentiometer_Bourns_3314J_Vertical
- R40: value 1k -> 22
- R43: value 10k -> 22
- R51: value 10k -> 1k
Connections:
- net labels added: +5V, D+, D-, FAN_MOSFET, PA13, PA14, PC_CONN
- net labels removed: BEEPER, E_STOP, FAN1_MOSFET, FAN2_MOSFET, KILL, RX, SPI_SS, TX
- wire segments 421 -> 445
Other:
- note added: "General considerations\nThe STM32 port currently requires an 8 MHz crystal for correct operation. The port is\ncurrently designed for and tested with STM32F103xB series MCUs, but it should work\nwith any STM32F103 series MCUs with minimal changes.\n\nUnlike Arduino-based boards, typically there is no automatic reset on serial connection\nwith STM32 boards. Please use restart_method: command with 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"
- note removed: "PA13, PA14 for debug! DONT USE"
- note removed: "use instead PA13 or PA14"

Commit message: change connection from USB to UART to support STM32 without USB
Parts:
- removed C49: 0u1, Capacitor_SMD:C_0603_1608Metric_Pad1.08x0.95mm_HandSolder, symbol Device:C
- removed D5: D_Schottky, Diode_SMD:D_SOD-323_HandSoldering, symbol Device:D_Schottky
- removed JP2: BOOT, Jumper:SolderJumper-2_P1.3mm_Open_TrianglePad1.0x1.5mm, symbol Jumper:Jumper_2_Open
- removed R43: 22, Resistor_SMD:R_0603_1608Metric_Pad0.98x0.95mm_HandSolder, symbol Device:R
- removed U8: USBLC6-2SC6, Package_TO_SOT_SMD:SOT-23-6, symbol Power_Protection:USBLC6-2SC6
- added C51, C52: 0u1, Capacitor_SMD:C_0603_1608Metric_Pad1.08x0.95mm_HandSolder, symbol Device:C
- added D5: LED, LED_SMD:LED_0603_1608Metric_Pad1.05x0.95mm_HandSolder, symbol Device:LED
- added U8: CH340E, Package_SO:MSOP-10_3x3mm_P0.5mm, symbol Interface_USB:CH340E
- R40: value 22 -> 1k
Connections:
- net labels added: RX, TX
- wire segments 445 -> 442
- no-connect marks 6 -> 7
Other:
- moved on the sheet: C50

Commit message: change PCB design
Parts:
- removed C50, C51, C52: 0u1, Capacitor_SMD:C_0603_1608Metric_Pad1.08x0.95mm_HandSolder, symbol Device:C
- removed D5: LED, LED_SMD:LED_0603_1608Metric_Pad1.05x0.95mm_HandSolder, symbol Device:LED
- removed R40: 1k, Resistor_SMD:R_0603_1608Metric_Pad0.98x0.95mm_HandSolder, symbol Device:R
- removed U2: STM32F103C8Tx, Package_QFP:LQFP-48_7x7mm_P0.5mm, symbol MCU_ST_STM32F1:STM32F103C8Tx
- removed U8: CH340E, Package_SO:MSOP-10_3x3mm_P0.5mm, symbol Interface_USB:CH340E
- added C3: 4u7, Capacitor_SMD:C_0603_1608Metric_Pad1.08x0.95mm_HandSolder, symbol Device:C
- added C35, C36: 1n, Capacitor_SMD:C_0603_1608Metric_Pad1.08x0.95mm_HandSolder, symbol Device:C
- added C41: 1u, Capacitor_SMD:C_0603_1608Metric_Pad1.08x0.95mm_HandSolder, symbol Device:C
- added J10: 5V, Connector_PinHeader_2.54mm:PinHeader_2x02_P2.54mm_Vertical, symbol Connector_Generic:Conn_02x02_Odd_Even
- added J16: Conn_01x06, Connector_PinHeader_2.54mm:PinHeader_1x06_P2.54mm_Vertical, symbol Connector_Generic:Conn_01x06
- added JP1: UART, Jumper:SolderJumper-2_P1.3mm_Open_TrianglePad1.0x1.5mm, symbol Device:Jumper_NC_Small
- added R1: 1m, Resistor_SMD:R_0603_1608Metric_Pad0.98x0.95mm_HandSolder, symbol Device:R
- added R10, R12, R14, R20, R21, R22, R23, R4, R6, R7, R8, R9: 10k, Resistor_SMD:R_0402_1005Metric_Pad0.72x0.64mm_HandSolder, symbol Device:R
- added U1: STM32F401CCUx, Package_DFN_QFN:QFN-48-1EP_7x7mm_P0.5mm_EP5.6x5.6mm, symbol MCU_ST_STM32F4:STM32F401CCUx
- added U8: USBLC6-2SC6, Package_TO_SOT_SMD:SOT-23-6, symbol Power_Protection:USBLC6-2SC6
- R11, R13, R15: footprint Resistor_SMD:R_0603_1608Metric_Pad0.98x0.95mm_HandSolder -> Resistor_SMD:R_0402_1005Metric_Pad0.72x0.64mm_HandSolder
- R16: renamed from R8; footprint Resistor_SMD:R_0603_1608Metric_Pad0.98x0.95mm_HandSolder -> Resistor_SMD:R_0402_1005Metric_Pad0.72x0.64mm_HandSolder
- R17: renamed from R10; footprint Resistor_SMD:R_0603_1608Metric_Pad0.98x0.95mm_HandSolder -> Resistor_SMD:R_0402_1005Metric_Pad0.72x0.64mm_HandSolder
- R18: renamed from R12; footprint Resistor_SMD:R_0603_1608Metric_Pad0.98x0.95mm_HandSolder -> Resistor_SMD:R_0402_1005Metric_Pad0.72x0.64mm_HandSolder
- R19: renamed from R14; footprint Resistor_SMD:R_0603_1608Metric_Pad0.98x0.95mm_HandSolder -> Resistor_SMD:R_0402_1005Metric_Pad0.72x0.64mm_HandSolder
- R28: renamed from R20; footprint Resistor_SMD:R_0603_1608Metric_Pad0.98x0.95mm_HandSolder -> Resistor_SMD:R_0402_1005Metric_Pad0.72x0.64mm_HandSolder
- R30: renamed from R22; footprint Resistor_SMD:R_0603_1608Metric_Pad0.98x0.95mm_HandSolder -> Resistor_SMD:R_0402_1005Metric_Pad0.72x0.64mm_HandSolder
- R32: renamed from R24; footprint Resistor_SMD:R_0603_1608Metric_Pad0.98x0.95mm_HandSolder -> Resistor_SMD:R_0402_1005Metric_Pad0.72x0.64mm_HandSolder
- R34: renamed from R26; footprint Resistor_SMD:R_0603_1608Metric_Pad0.98x0.95mm_HandSolder -> Resistor_SMD:R_0402_1005Metric_Pad0.72x0.64mm_HandSolder
- R5: renamed from R9; footprint Resistor_SMD:R_0603_1608Metric_Pad0.98x0.95mm_HandSolder -> Resistor_SMD:R_0402_1005Metric_Pad0.72x0.64mm_HandSolder
- renumbered C17 to C10, C18 to C11, C19 to C12, C20 to C13, C21 to C14, C22 to C15, C23 to C16, C24 to C17, C25 to C18, C26 to C19, C27 to C20, C28 to C21, C29 to C22, C30 to C23, C31 to C24, C32 to C25, C33 to C26, C34 to C27, C35 to C28, C36 to C29, C37 to C30, C38 to C31, C39 to C32, C40 to C33, C7 to C34, C9 to C37, C3 to C38, C10 to C39, C11 to C40, C6 to C42, C8 to C43, C48 to C44, C12 to C45, C43 to C46, C44 to C47, C41 to C48, C42 to C49, C45 to C50, C46 to C51, C47 to C52, C13 to C6, C14 to C7, C15 to C8, C16 to C9, D6 to D4, D4 to D5, D7 to D6, J2 to J1, J1 to J2, J5 to J4, J8 to J5, J9 to J6, J6 to J7, J10 to J8, J7 to J9, Q5 to Q4, Q6 to Q5, R52 to R2, R16 to R24, R17 to R25, R18 to R26, R19 to R27, R21 to R29, R53 to R3, R23 to R31, R25 to R33, R27 to R35, R28 to R36, R29 to R37, R30 to R38, R31 to R39, R32 to R40, R33 to R41, R34 to R42, R35 to R43, R1 to R44, R2 to R45, R3 to R46, R4 to R47, R5 to R48, R51 to R49, R54 to R50, R6 to R51, R7 to R52, R45 to R53, R46 to R54, R36 to R55, R37 to R56, R38 to R57, R39 to R58, R41 to R59, R42 to R60, R44 to R61, R47 to R62, R48 to R63, R49 to R64, R50 to R65, U4 to U2, U5 to U3, U6 to U4, U7 to U5, U3 to U6, U1 to U7
Connections:
- net labels added: CS, CS1, CS2, PH0, PH1, USB_DM, USB_DP, VCAP
- net labels removed: RX, SCL, SDA, TX
- wire segments 442 -> 447
- no-connect marks 7 -> 6
Other:
- note removed: "General considerations\nThe STM32 port currently requires an 8 MHz crystal for correct operation. The port is\ncurrently designed for and tested with STM32F103xB series MCUs, but it should work\nwith any STM32F103 series MCUs with minimal changes.\n\nUnlike Arduino-based boards, typically there is no automatic reset on serial connection\nwith STM32 boards. Please use restart_method: command with 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"
- moved on the sheet: C1, C10, C11, C12, C13, C14, C15, C16, C17, C18, C19, C2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

Commit message: pcb fixes
Parts:
- removed J16: Conn_01x06, Connector_PinHeader_2.54mm:PinHeader_1x06_P2.54mm_Vertical, symbol Connector_Generic:Conn_01x06
- C10, C11, C12, C13: value 0u22 -> 2u2
- C14, C15, C16, C17: value 0u1 -> 22n
- C45, L1: value 10u -> 22u
- C6, C7, C8, C9: value 0u22 -> 0u1
- D5: value D_Schottky -> SS34
- R24, R25, R26, R27: value R* -> 10k
- R29, R31, R33, R35: value R* -> 10k; footprint Potentiometer_SMD:Potentiometer_Bourns_3314J_Vertical -> Potentiometer_SMD:Potentiometer_Bourns_TC33X_Vertical
- R51: value R -> 210k
- R52: value R -> 40k2
Other:
- moved on the sheet: C45, D5, L1, R51, R52
